Commit message: changes

File: chipta_bot/urdf/chipta.xacro (robot description, xacro)
@@ -35,5 +35,5 @@
       <mesh filename="file://$(find chipta_bot)/meshes/IMU_v1_1.stl" scale="0.001 0.001 0.001"/>
     </geometry>
-    <material name="silver"/>
+    <material name="light_blue"/>
   </visual>
   <collision>
@@ -55,5 +55,5 @@
       <mesh filename="file://$(find chipta_bot)/meshes/GPS_v1_1.stl" scale="0.001 0.001 0.001"/>
     </geometry>
-    <material name="silver"/>
+    <material name="green"/>
   </visual>
   <collision>
@@ -75,5 +75,5 @@
       <mesh filename="file://$(find chipta_bot)/meshes/Lidar_v1_1.stl" scale="0.001 0.001 0.001"/>
     </geometry>
-    <material name="silver"/>
+    <material name="blue"/>
   </visual>
   <collision>

File: chipta_bot/urdf/materials.xacro (robot description, xacro)
@@ -5,8 +5,17 @@
 </material>
 <material name="purple">
-  <color rgba="0.5 0.0 0.7 1.0"/>
+  <color rgba="0.6 0.3 0.8 1.0"/>
 </material>
 <material name="black">
   <color rgba="0 0 0 1"/>
 </material>
+<material name="blue">
+  <color rgba="0 0 0.9 1"/>
+</material>
+<material name="light_blue">
+  <color rgba="0.4 0.7 1.0 1.0"/>
+</material>
+<material name="green">
+  <color rgba="0.2 0.8 0.2 1.0"/>
+</material>
 </robot>
