Commit message: mecanum plugin

File: helios_description/urdf/helios_description.xacro (robot description, xacro)
@@ -179,5 +179,5 @@
   <child link="Lidar_v1_1"/>
 </joint>
-<joint name="Revolute 24" type="continuous">
+<joint name="wheel_front_left_joint" type="continuous">
   <origin xyz="0.064778 0.085 0.030131" rpy="0 0 0"/>
   <parent link="base_link"/>
@@ -185,5 +185,5 @@
   <axis xyz="0.0 1.0 0.0"/>
 </joint>
-<joint name="Revolute 25" type="continuous">
+<joint name="wheel_front_right_joint" type="continuous">
   <origin xyz="0.064778 -0.085 0.030131" rpy="0 0 0"/>
   <parent link="base_link"/>
@@ -191,5 +191,5 @@
   <axis xyz="0.0 -1.0 0.0"/>
 </joint>
-<joint name="Revolute 27" type="continuous">
+<joint name="wheel_rear_right_joint" type="continuous">
   <origin xyz="-0.064941 -0.085 0.031781" rpy="0 0 0"/>
   <parent link="base_link"/>
@@ -197,5 +197,5 @@
   <axis xyz="0.0 1.0 0.0"/>
 </joint>
-<joint name="Revolute 28" type="continuous">
+<joint name="wheel_rear_left_joint" type="continuous">
   <origin xyz="-0.064941 0.085 0.030131" rpy="0 0 0"/>
   <parent link="base_link"/>
